File: circuit/candle_circuit.brd (EAGLE design)
At the start: 37.8 x 53.3 mm, 21 parts, among them IC1 TINY10P, SW1 KMR2, SW2 KMR2, X1 ESP-12

Commit message: Circuit board updates
Parts:
- removed D3: MBR120, microbuilder:SOD-123
- added D1: MBR120, microbuilder:SOD-123
- added R7, R8: 10K, microbuilder:0805-NO
- LED1: device adafruit:CHIPLED_0603 -> microbuilder:CHIPLED_0805_NOOUTLINE
- R1: value 10k -> 1k
- R3: value 1M -> 10k
- R5: value 10k -> 1M
- moved R3 43.9 mm to (12.7, 1.78), turned to 0 degrees
- moved R5 43.9 mm to (22.9, 44.5), turned to 270 degrees
- moved C1 14.0 mm to (33.0, 3.81)
- moved C2 14.0 mm to (33.0, 17.8)
- moved R1 9.21 mm to (26.7, 10.2)
- moved LED1 6.10 mm to (26.9, 7.87), turned to 90 degrees
- moved JP2 3.66 mm to (28.7, 47.5)
- moved SW1 2.54 mm to (26.7, 3.81)
- renumbered R4 to R6
Connections:
- new net GPIO2: R8.1, X1.11
- new net N$6: LED1.C, R1.1
- net +3V3: now also LED1.A, R3.1, R8.2; no longer R1.2, R5.1
- net CH_PD: now also R3.2; no longer R5.2
- net GND: now also R7.1; no longer LED1.C
- net GPIO0: now also R1.2
- net GPIO15: now also R7.2, X1.10; no longer IC1.1, X1.13
- net N$4: now also IC1.1, X1.13; no longer LED1.A, R1.1
- net N$5: now also D1.C; no longer D3.C
- net N$7: now also R5.2; no longer R3.2
- net SENSOR: now also R5.1; no longer R3.1
- net V+: now also D1.A; no longer D3.A
Routing:
- net +3V3: track 46.2 -> 85.3 mm
- net N$4: track 2.21 -> 24.3 mm
- net GPIO15: track 23.9 -> 2.92 mm
- net GND: track 145.0 -> 134.9 mm
- net GPIO2: track 0.00 -> 5.97 mm
- net N$6: track 0.00 -> 2.82 mm
- net SENSOR: track 19.6 -> 22.0 mm
- net GPIO0: track 11.6 -> 13.3 mm
- net V+: track 63.3 -> 61.7 mm
- net RXD: track 8.83 -> 7.20 mm
