File: circuit/candle_circuit.brd (EAGLE design)
At the start: 37.8 x 53.3 mm, 25 parts, among them IC1 TINY10P, SW1 KMR2, SW2 KMR2, X1 ESP-12

Commit message: Board updates
Parts:
- JP5: value Test -> TEST; device microbuilder:1X02_OVAL -> pinhead:1X01
- moved JP5 25.2 mm to (16.5, 1.02), turned to 0 degrees
- moved JP4 1.27 mm to (33.0, 29.0)
Connections:
- net +3V3: now also JP5.1; no longer JP5.2
- net GND: no longer JP5.1
Routing:
- net V+: track 61.7 -> 66.4 mm
- net GND: track 130.5 -> 126.2 mm
- net +3V3: track 85.8 -> 86.3 mm
Changed lines of the file:
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@@
 <element name="R5" library="adafruit" package="R0603" value="10k" x="20.828" y="22.098"/>
 <element name="R4" library="adafruit" package="R0603" value="10k" x="15.748" y="23.114"/>
-<element name="JP4" library="microbuilder" package="1X02_OVAL" value="Test" x="33.02" y="30.226" rot="R180"/>
-<element name="JP5" library="microbuilder" package="1X02_OVAL" value="Test" x="41.656" y="0.508" rot="R180"/>
+<element name="JP4" library="microbuilder" package="1X02_OVAL" value="Test" x="33.02" y="28.956" rot="R180"/>
+<element name="JP5" library="pinhead" package="1X01" value="TEST" x="16.51" y="1.016"/>
 </elements>
 <signals>
@@
 <wire x1="8.128" y1="50.546" x2="30.48" y2="50.546" width="0.6096" layer="1"/>
 <wire x1="30.48" y1="50.546" x2="34.29" y2="46.99" width="0.6096" layer="1"/>
-<wire x1="34.29" y1="46.99" x2="34.29" y2="24.13" width="0.6096" layer="1"/>
-<wire x1="24.04" y1="30.1" x2="25.69" y2="31.75" width="0.6096" layer="1"/>
-<wire x1="25.69" y1="31.75" x2="31.75" y2="31.75" width="0.6096" layer="1"/>
-<wire x1="31.75" y1="31.75" x2="34.29" y2="29.21" width="0.6096" layer="1"/>
-<wire x1="34.29" y1="29.21" x2="34.29" y2="24.13" width="0.6096" layer="1"/>
+<wire x1="34.29" y1="46.99" x2="34.29" y2="32.004" width="0.6096" layer="1"/>
+<wire x1="24.04" y1="30.1" x2="27.214" y2="34.036" width="0.6096" layer="1"/>
+<wire x1="27.214" y1="34.036" x2="31.496" y2="34.036" width="0.6096" layer="1"/>
+<wire x1="31.496" y1="34.036" x2="34.29" y2="32.004" width="0.6096" layer="1"/>
+<wire x1="34.29" y1="32.004" x2="34.29" y2="24.13" width="0.6096" layer="1"/>
 <wire x1="19.05" y1="38.1" x2="19.05" y2="36.83" width="0.6096" layer="1"/>
 <wire x1="19.05" y1="36.83" x2="21.59" y2="34.29" width="0.6096" layer="1"/>
@@
 <contactref element="R5" pad="2"/>
 <contactref element="JP4" pad="1"/>
-<contactref element="JP5" pad="1"/>
-<wire x1="35.87" y1="5.06" x2="42.926" y2="0.508" width="0" layer="19" extent="1-1"/>
 <wire x1="27.47" y1="5.86" x2="27.488" y2="1.778" width="0" layer="19" extent="1-1"/>
 <wire x1="21.082" y1="25.616" x2="24.04" y2="30.1" width="0" layer="19" extent="1-1"/>
@@
 <wire x1="11.85" y1="1.778" x2="11.85" y2="1.358" width="0.6096" layer="1"/>
 <wire x1="11.85" y1="1.358" x2="12.7" y2="0.254" width="0.6096" layer="1"/>
-<wire x1="12.7" y1="0.254" x2="21.336" y2="0.254" width="0.6096" layer="1"/>
+<wire x1="12.7" y1="0.254" x2="15.748" y2="0.254" width="0.6096" layer="1"/>
+<wire x1="15.748" y1="0.254" x2="16.51" y2="1.016" width="0.6096" layer="1"/>
+<wire x1="17.526" y1="0.254" x2="21.336" y2="0.254" width="0.6096" layer="1"/>
 <wire x1="21.336" y1="0.254" x2="22.987" y2="1.905" width="0.6096" layer="1"/>
 <wire x1="22.987" y1="1.905" x2="23.241" y2="1.905" width="0.6096" layer="1"/>
@@
 <wire x1="14.898" y1="23.114" x2="13.716" y2="23.114" width="0.4064" layer="1"/>
 <wire x1="13.716" y1="23.114" x2="13.462" y2="23.368" width="0.4064" layer="1"/>
-<contactref element="JP5" pad="2"/>
-<wire x1="31.75" y1="3.81" x2="40.386" y2="0.508" width="0" layer="19" extent="1-1"/>
-<wire x1="30.48" y1="8.89" x2="29.92" y2="9.13" width="0" layer="19" extent="1-1"/>
+<contactref element="JP5" pad="1"/>
+<wire x1="16.51" y1="1.016" x2="17.526" y2="0.254" width="0.6096" layer="1"/>
+<wire x1="29.92" y1="9.13" x2="30.48" y2="8.89" width="0" layer="19" extent="1-1"/>
 </signal>
 <signal name="V+">
@@
 <wire x1="27.0002" y1="28.8798" x2="31.75" y2="24.13" width="0.6096" layer="1"/>
 <contactref element="JP4" pad="2"/>
-<wire x1="27.0002" y1="28.8798" x2="31.75" y2="30.226" width="0" layer="19" extent="1-1"/>
+<wire x1="27.0002" y1="28.8798" x2="31.75" y2="28.956" width="0.6096" layer="1"/>
 </signal>
 <signal name="N$1">

Commit message: Updates to board and schematic
Parts:
- JP1: value FTDI -> Serial
- JP4: value Test -> V+ Test
- JP5: value TEST -> 3V3 Test
- renumbered U$1 to U1, X1 to IC2
